File: benboard/benboard.kicad_pcb (KiCad board)
At the start: 2 copper layers, 59 parts, among them J1 USB_C_Receptacle_USB2.0, SW1 SW_Push, SW10 SW_Push, SW11 SW_Push, SW12 SW_Push, SW13 SW_Push, SW14 SW_Push, SW15 SW_Push, SW16 SW_Push, SW17 SW_Push, SW18 SW_Push, SW19 SW_Push, SW2 SW_Push, SW20 SW_Push, SW21 SW_Push, SW3 SW_Push, SW4 SW_Push, SW5 SW_Push, SW6 SW_Push, SW7 SW_Push, SW8 SW_Push, SW9 SW_Push, U1 nRF52840, U2 BQ24075RGT, Y1 32MHz, Y2 32.768kHz

Commit message: awesome
Parts:
- added REF**: SW_Cherry_MX_1.00u_PCB, Button_Switch_Keyboard:SW_Cherry_MX_1.00u_PCB, F.Cu at (132.5, 66.9)
- added REF**: SW_Cherry_MX_1.00u_PCB, Button_Switch_Keyboard:SW_Cherry_MX_1.00u_PCB, F.Cu at (151.6, 68.0)
- added REF**: SW_Cherry_MX_1.00u_PCB, Button_Switch_Keyboard:SW_Cherry_MX_1.00u_PCB, F.Cu at (170.7, 49.9)
- added REF**: SW_Cherry_MX_1.00u_PCB, Button_Switch_Keyboard:SW_Cherry_MX_1.00u_PCB, F.Cu at (170.7, 88.0)
- added REF**: SW_Cherry_MX_1.00u_PCB, Button_Switch_Keyboard:SW_Cherry_MX_1.00u_PCB, F.Cu at (113.5, 88.2)
- added REF**: SW_Cherry_MX_1.00u_PCB, Button_Switch_Keyboard:SW_Cherry_MX_1.00u_PCB, F.Cu at (170.7, 69.0)
- added REF**: SW_Cherry_MX_1.00u_PCB, Button_Switch_Keyboard:SW_Cherry_MX_1.00u_PCB, F.Cu at (113.5, 69.1)
- added REF**: SW_Cherry_MX_1.00u_PCB, Button_Switch_Keyboard:SW_Cherry_MX_1.00u_PCB, F.Cu at (180.0, 109.5)
- added REF**: SW_Cherry_MX_1.00u_PCB, Button_Switch_Keyboard:SW_Cherry_MX_1.00u_PCB, F.Cu at (157.0, 107.4)
- added REF**: SW_Cherry_MX_1.00u_PCB, Button_Switch_Keyboard:SW_Cherry_MX_1.00u_PCB, F.Cu at (75.3, 76.9)
- added REF**: SW_Cherry_MX_1.00u_PCB, Button_Switch_Keyboard:SW_Cherry_MX_1.00u_PCB, F.Cu at (94.3, 53.4)
- added REF**: SW_Cherry_MX_1.00u_PCB, Button_Switch_Keyboard:SW_Cherry_MX_1.00u_PCB, F.Cu at (94.3, 91.5)
- added REF**: SW_Cherry_MX_1.00u_PCB, Button_Switch_Keyboard:SW_Cherry_MX_1.00u_PCB, F.Cu at (113.5, 50.0)
- added REF**: SW_Cherry_MX_1.00u_PCB, Button_Switch_Keyboard:SW_Cherry_MX_1.00u_PCB, F.Cu at (151.6, 87.1)
- added REF**: SW_Cherry_MX_1.00u_PCB, Button_Switch_Keyboard:SW_Cherry_MX_1.00u_PCB, F.Cu at (151.6, 48.9)
- added REF**: SW_Cherry_MX_1.00u_PCB, Button_Switch_Keyboard:SW_Cherry_MX_1.00u_PCB, F.Cu at (132.5, 47.8)
- added REF**: SW_Cherry_MX_1.00u_PCB, Button_Switch_Keyboard:SW_Cherry_MX_1.00u_PCB, F.Cu at (201.2, 114.8)
- added REF**: SW_Cherry_MX_1.00u_PCB, Button_Switch_Keyboard:SW_Cherry_MX_1.00u_PCB, F.Cu at (75.3, 57.8)
- added REF**: SW_Cherry_MX_1.00u_PCB, Button_Switch_Keyboard:SW_Cherry_MX_1.00u_PCB, F.Cu at (94.3, 72.5)
- added REF**: SW_Cherry_MX_1.00u_PCB, Button_Switch_Keyboard:SW_Cherry_MX_1.00u_PCB, F.Cu at (132.5, 86.0)
- added REF**: SW_Cherry_MX_1.00u_PCB, Button_Switch_Keyboard:SW_Cherry_MX_1.00u_PCB, F.Cu at (75.3, 96.0)
- C1, C10, C11, C12, C13, C14, C15, C16, C17, C18, C19, C2, C20, C21, C22, C23, C3, C4, C5, C6, C7, C8, C9, J1, L1, L2, L3, L4, R1, R2, R3, R4, R5, RED1, U1, U2, Y1, Y2: moved to B.Cu
- moved C18 66.1 mm to (144.4, 109.6), turned to -45 degrees
- moved SW19 61.4 mm to (154.5, 112.5)
- moved R5 55.6 mm to (235.1, 68.5), turned to 180 degrees
- moved R3 55.6 mm to (235.1, 65.8), turned to 180 degrees
- moved L1 52.4 mm to (231.5, 65.1), turned to 0 degrees
- moved SW16 51.6 mm to (168.1, 55.0)
- moved U2 48.5 mm to (227.0, 66.4), turned to 180 degrees
- moved R1 47.6 mm to (159.1, 48.8), turned to 180 degrees
- moved U1 46.7 mm to (145.2, 103.8), turned to 135 degrees
- moved SW20 46.5 mm to (176.8, 114.2), turned to -8 degrees
- moved SW21 45.3 mm to (197.4, 119.0), turned to -16 degrees
- moved C3 44.6 mm to (226.0, 69.9), turned to 180 degrees
- moved R2 41.9 mm to (167.4, 47.0), turned to -90 degrees
- moved RED1 40.4 mm to (222.8, 68.1)
- moved Y2 38.0 mm to (214.8, 69.8)
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Connections:
- C1 pad 2: VBAT -> GND
- C10 pad 2: VBAT -> GND
- C11 pad 2: VBAT -> GND
- C12 pad 2: VBAT -> GND
- C13 pad 2: VBAT -> GND
- C14 pad 2: VBAT -> GND
- C15 pad 2: VBAT -> GND
- C16 pad 1: VBAT -> GND
- C17 pad 1: VBAT -> GND
- C18 pad 2: VBAT -> GND
- C19 pad 2: VBAT -> GND
- C2 pad 2: VBAT -> GND
- C20 pad 2: Net-(C20-Pad2) -> GND
- C21 pad 2: VBAT -> GND
- C22 pad 1: VBAT -> GND
- C23 pad 1: VBAT -> GND
- C3 pad 2: VBAT -> GND
- C4 pad 2: VBAT -> GND
- C5 pad 2: VBAT -> GND
- C6 pad 2: VBAT -> GND
- C7 pad 2: VBAT -> GND
- C8 pad 2: VBAT -> GND
- C9 pad 2: VBAT -> GND
- J1 pad A1: VBAT -> GND
- J1 pad A12: VBAT -> GND
- J1 pad A4: Net-(J1-VBUS-PadA4) -> VBUS
- J1 pad A9: Net-(J1-VBUS-PadA4) -> VBUS
- J1 pad B1: VBAT -> GND
- J1 pad B12: VBAT -> GND
- J1 pad B4: Net-(J1-VBUS-PadA4) -> VBUS
- J1 pad B9: Net-(J1-VBUS-PadA4) -> VBUS
- R1 pad 2: VBAT -> GND
- R2 pad 2: VBAT -> GND
- R4 pad 2: VBAT -> GND
- R5 pad 1: VBAT -> GND
- U1 pad B7: VBAT -> GND
- U1 pad EP: VBAT -> GND
- U1 pad F23: VBAT -> GND
- U2 pad 15: VBAT -> GND
- U2 pad 17: VBAT -> GND
- U2 pad 2: Net-(C20-Pad2) -> VBAT
- U2 pad 3: Net-(C20-Pad2) -> VBAT
- U2 pad 4: VBAT -> GND
- U2 pad 5: VBAT -> GND
- U2 pad 8: VBAT -> GND
- Y1 pad 2: VBAT -> GND
- Y2 pad 2: VBAT -> GND
Routing:
- net Net-(J1-CC2): track 0.00 -> 11.1 mm, vias 0 -> 2
- net VBUS: track 0.00 -> 8.34 mm
- net unconnected-(U1-NFC1/P0.09-PadL24): track 0.00 -> 7.86 mm
- net unconnected-(U1-NFC2/P0.10-PadJ24): track 0.00 -> 7.86 mm
- net unconnected-(U1-P0.20-PadAD16): track 0.00 -> 7.49 mm
- net Net-(U1-DEC5): track 0.00 -> 7.45 mm
- net unconnected-(U1-P1.06-PadR24): track 0.00 -> 7.05 mm
- net unconnected-(U1-P1.04-PadU24): track 0.00 -> 6.66 mm
- net unconnected-(U1-TRACEDATA0/P1.00-PadAD22): track 0.00 -> 6.56 mm
- net unconnected-(U1-P1.02-PadW24): track 0.00 -> 6.27 mm
- net VDD_NRF: track 0.00 -> 6.12 mm
- net unconnected-(U1-P0.24-PadAD20): track 0.00 -> 5.90 mm
- net SWDC: track 0.00 -> 5.87 mm
- net unconnected-(U1-P0.22-PadAD18): track 0.00 -> 5.70 mm
- net SWDI: track 0.00 -> 5.68 mm
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Other:
- board outline added: 150.3 x 92.1 mm
- copper layers 2 -> 4

Commit message: epic
Parts:
- removed C15: 100pF, Capacitor_SMD:C_0603_1608Metric
- removed REF** (x21): SW_Cherry_MX_1.00u_PCB, Button_Switch_Keyboard:SW_Cherry_MX_1.00u_PCB
- C14: value 100pF -> 0.5pF; moved to F.Cu
- C21: value 100pF -> 0.8pF; moved to F.Cu
- L4: value 3.9nH -> 4.1nH; moved to F.Cu
- R3, RED1: moved to F.Cu
- SW1, SW10, SW11, SW12, SW13, SW14, SW15, SW16, SW17, SW18, SW19, SW2, SW20, SW21, SW3, SW4, SW5, SW6, SW7, SW8, SW9: footprint keyswitches:Kailh_socket_MX_optional_reversible -> keyswitches:Kailh_socket_MX
- moved C12 92.1 mm to (131.2, 86.6), turned to -90 degrees
- moved C10 90.7 mm to (132.8, 83.6), turned to 90 degrees
- moved C9 89.1 mm to (131.2, 83.6), turned to 90 degrees
- moved L1 86.6 mm to (147.0, 84.0), turned to 180 degrees
- moved L3 86.2 mm to (134.4, 83.6), turned to -90 degrees
- moved C11 85.4 mm to (134.4, 86.6), turned to -90 degrees
- moved C5 80.5 mm to (134.6, 80.4)
- moved C22 79.9 mm to (139.9, 96.5), turned to 90 degrees
- moved Y2 77.4 mm to (140.9, 92.8)
- moved C6 75.9 mm to (138.4, 90.6), turned to -90 degrees
- moved C3 74.4 mm to (153.0, 84.0), turned to 0 degrees
- moved C23 72.8 mm to (144.3, 90.2)
- moved R3 72.4 mm to (165.3, 46.6)
- moved L4 71.1 mm to (149.0, 81.8)
- moved C13 70.3 mm to (132.8, 86.6), turned to -90 degrees
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Connections:
- J1 pad S1: unconnected-(J1-SHIELD-PadS1) -> GND
- SW1 pad 1: unconnected-(SW1-Pad1) -> GND
- SW1 pad 2: unconnected-(SW1-Pad2) -> SW1
- SW10 pad 1: unconnected-(SW10-Pad1) -> GND
- SW10 pad 2: unconnected-(SW10-Pad2) -> SW10
- SW11 pad 1: unconnected-(SW11-Pad1) -> GND
- SW11 pad 2: unconnected-(SW11-Pad2) -> SW11
- SW12 pad 1: unconnected-(SW12-Pad1) -> GND
- SW12 pad 2: unconnected-(SW12-Pad2) -> SW12
- SW13 pad 1: unconnected-(SW13-Pad1) -> GND
- SW13 pad 2: unconnected-(SW13-Pad2) -> SW13
- SW14 pad 1: unconnected-(SW14-Pad1) -> GND
- SW14 pad 2: unconnected-(SW14-Pad2) -> SW14
- SW15 pad 1: unconnected-(SW15-Pad1) -> GND
- SW15 pad 2: unconnected-(SW15-Pad2) -> SW15
- SW16 pad 1: unconnected-(SW16-Pad1) -> GND
- SW16 pad 2: unconnected-(SW16-Pad2) -> SW16
- SW17 pad 1: unconnected-(SW17-Pad1) -> GND
- SW17 pad 2: unconnected-(SW17-Pad2) -> SW17
- SW18 pad 1: unconnected-(SW18-Pad1) -> GND
- SW18 pad 2: unconnected-(SW18-Pad2) -> SW18
- SW19 pad 1: unconnected-(SW19-Pad1) -> GND
- SW19 pad 2: unconnected-(SW19-Pad2) -> SW19
- SW2 pad 1: unconnected-(SW2-Pad1) -> GND
- SW2 pad 2: unconnected-(SW2-Pad2) -> SW2
- SW20 pad 1: unconnected-(SW20-Pad1) -> GND
- SW20 pad 2: unconnected-(SW20-Pad2) -> SW20
- SW21 pad 1: unconnected-(SW21-Pad1) -> GND
- SW21 pad 2: unconnected-(SW21-Pad2) -> SW21
- SW3 pad 1: unconnected-(SW3-Pad1) -> GND
- SW3 pad 2: unconnected-(SW3-Pad2) -> SW3
- SW4 pad 1: unconnected-(SW4-Pad1) -> GND
- SW4 pad 2: unconnected-(SW4-Pad2) -> SW4
- SW5 pad 1: unconnected-(SW5-Pad1) -> GND
- SW5 pad 2: unconnected-(SW5-Pad2) -> SW5
- SW6 pad 1: unconnected-(SW6-Pad1) -> GND
- SW6 pad 2: unconnected-(SW6-Pad2) -> SW6
- SW7 pad 1: unconnected-(SW7-Pad1) -> GND
- SW7 pad 2: unconnected-(SW7-Pad2) -> SW7
- SW8 pad 1: unconnected-(SW8-Pad1) -> GND
- SW8 pad 2: unconnected-(SW8-Pad2) -> SW8
- SW9 pad 1: unconnected-(SW9-Pad1) -> GND
- SW9 pad 2: unconnected-(SW9-Pad2) -> SW9
- U1 pad AC15: unconnected-(U1-P0.19-PadAC15) -> SW2
- U1 pad AC17: unconnected-(U1-P0.21-PadAC17) -> SW5
- U1 pad AC19: unconnected-(U1-P0.23-PadAC19) -> SW8
- U1 pad AC21: unconnected-(U1-P0.25-PadAC21) -> SW11
- U1 pad AD10: unconnected-(U1-P0.15-PadAD10) -> SW1
- U1 pad AD12: unconnected-(U1-P0.17-PadAD12) -> SW4
- U1 pad AD16: unconnected-(U1-P0.20-PadAD16) -> SW7
- U1 pad AD18: unconnected-(U1-P0.22-PadAD18) -> SW10
- U1 pad AD20: unconnected-(U1-P0.24-PadAD20) -> SW13
- U1 pad AD22: unconnected-(U1-TRACEDATA0/P1.00-PadAD22) -> SW14
- U1 pad H2: unconnected-(U1-P0.27-PadH2) -> SW12
- U1 pad L1: unconnected-(U1-P0.06-PadL1) -> SW9
- U1 pad N1: unconnected-(U1-P0.08-PadN1) -> SW6
- U1 pad P2: unconnected-(U1-P1.08-PadP2) -> SW3
- U1 pad P23: unconnected-(U1-P1.07-PadP23) -> SW15
- U1 pad R24: unconnected-(U1-P1.06-PadR24) -> SW18
- U1 pad T23: unconnected-(U1-P1.05-PadT23) -> SW21
- U1 pad U24: unconnected-(U1-P1.04-PadU24) -> SW17
- U1 pad V23: unconnected-(U1-P1.03-PadV23) -> SW20
- U1 pad W24: unconnected-(U1-P1.02-PadW24) -> SW16
- U1 pad Y23: unconnected-(U1-P1.01-PadY23) -> SW19
Routing:
- net VBUS: track 8.34 -> 119.4 mm, vias 0 -> 5
- net GND: track 3.67 -> 97.4 mm, vias 0 -> 25
- net VDDH: track 0.00 -> 89.3 mm, vias 0 -> 6
- net SW21: track 0.00 -> 87.1 mm, vias 0 -> 2
- net SW1: track 0.00 -> 82.4 mm
- net SW3: track 0.00 -> 78.4 mm, vias 0 -> 2
- net D-: track 2.70 -> 71.9 mm, vias 0 -> 2
- net D+: track 2.84 -> 71.3 mm, vias 0 -> 2
- net SW4: track 0.00 -> 67.7 mm
- net SW20: track 0.00 -> 67.6 mm, vias 0 -> 2
- net SW2: track 0.00 -> 62.3 mm, vias 0 -> 2
- net Net-(RED1-K): track 0.00 -> 56.7 mm, vias 0 -> 4
- net SW6: track 0.00 -> 56.2 mm
- net SW16: track 0.00 -> 50.1 mm
- net SW18: track 0.00 -> 49.6 mm
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- added copper zone on B.Cu, net GND
- added copper zone on F.Cu, net GND
- added copper zone on In1.Cu, net GND
- added copper zone on In2.Cu, net GND
Other:
- board size 150.3 x 92.1 mm -> 140 x 88.4 mm
- board text added: "- SWD - RESET / POWER BUTTON - ESD PROTECTION - BATTERY PADS - PROBE POINTS - ANT JUMPERS"
- board text added: "0.1 DEVEL"
- board text added: "Ben Labs"
- board text added: "BenBoard"
- board text added: "PCB3D_BR_BENBOARD"
- board text added: "PCB3D_TL_BENBOARD"
