File: benboard/benboard.kicad_sch (KiCad schematic)
At the start: 1 part, among them U1 nRF52840

Commit message: keyboad
Parts:
- added C1, C19, C2, C20, C5, C9: 4.7uF, Capacitor_SMD:C_0603_1608Metric, symbol Device:C
- added C10, C11, C12, C6: 100nF, Capacitor_SMD:C_0603_1608Metric, symbol Device:C
- added C13, C18, C3: 1uF, Capacitor_SMD:C_0603_1608Metric, symbol Device:C
- added C14, C15, C21, C7: 100pF, Capacitor_SMD:C_0603_1608Metric, symbol Device:C
- added C16, C17, C22, C23: 12pF, Capacitor_SMD:C_0603_1608Metric, symbol Device:C
- added C4: 47nF, Capacitor_SMD:C_0603_1608Metric, symbol Device:C
- added C8: 820pF, Capacitor_SMD:C_0603_1608Metric, symbol Device:C
- added J1: USB_C_Receptacle_USB2.0, Connector_USB:USB_C_Receptacle_G-Switch_GT-USB-7010ASV, symbol Connector:USB_C_Receptacle_USB2.0
- added L1, L3: 10uH, Inductor_SMD:L_0603_1608Metric, symbol Device:L
- added L2: 15nH, Inductor_SMD:L_0603_1608Metric, symbol Device:L
- added L4: 3.9nH, Inductor_SMD:L_0603_1608Metric, symbol Device:L
- added R1, R2: 5.1k, Resistor_SMD:R_0603_1608Metric, symbol Device:R
- added R3, R4, R5: 10k, Resistor_SMD:R_0603_1608Metric, symbol Device:R
- added RED1: LED, LED_SMD:LED_0805_2012Metric, symbol Device:LED
- added SW1 (x21): SW_Push, keyswitches:Kailh_socket_MX_optional_reversible, symbol Switch:SW_Push
- added U2: BQ24075RGT, Package_DFN_QFN:VQFN-16-1EP_3x3mm_P0.5mm_EP1.6x1.6mm, symbol Battery_Management:BQ24075RGT
- added Y1: 32MHz, Crystal:Crystal_SMD_SeikoEpson_FA238V-4Pin_3.2x2.5mm, symbol Device:Crystal_GND2
- added Y2: 32.768kHz, Crystal:Crystal_SMD_SeikoEpson_FA238V-4Pin_3.2x2.5mm, symbol Device:Crystal_GND2
Connections:
- net VDD_NRF: now reaches U1.A22 (VDD), U1.AD14 (VDD), U1.AD23 (VDD), U1.B1 (VDD), U1.W1 (VDD)
- net VDD_NRF: now also C10.1, C11.1, C12.1, C13.1, C9.1, L3.2
- net at U1.A23 (XC2): now also C17.2, Y1.3
- net SWDC: now reaches U1.AA24 (SWDCLK)
- net at U1.AB2 (DCCH): now also L3.1
- net RST: now reaches U1.AC11 (P0.16)
- net RST: now also U1.AC13 (P0.18/~{RESET}), U1.AC9 (P0.14)
- net SWDI: now reaches U1.AC24 (SWDIO)
- net at U1.AC5 (DECUSB): now also C5.1
- net VBUS: now reaches U1.AD2 (VBUS)
- net VBUS: now also C1.1, C18.1, U2.13 (IN)
- net D-: now reaches U1.AD4 (D-)
- net D-: now also J1.A7 (D-), J1.B7 (D-)
- net D+: now reaches U1.AD6 (D+)
- net D+: now also J1.A6 (D+), J1.B6 (D+)
- net POWER: now reaches U1.AD8 (P0.13)
- net at U1.B24 (XC1): now also C16.2, Y1.1
- net at U1.B3 (DCC): now also L1.2
- net at U1.B5 (DEC4): now also U1.E24 (DEC6), C3.1, C4.1, L2.1
- net GND: now reaches U1.B7 (VSS), U1.EP (VSS)
- net GND: now also U1.F23 (VSS_PA), C1.2, C10.2, C11.2, C12.2, C13.2, C14.2, C15.2, C16.1, C17.1, C18.2, C19.2, C2.2, C20.1, C21.2, C22.1, C23.1, C3.2, C4.2, C5.2, C6.2, C7.2, C8.2, C9.2, J1.A1 (GND), J1.A12 (GND), J1.B1 (GND), J1.B12 (GND), R1.2, R2.2, R4.2, R5.1, U2.15 (SYSOFF), U2.17 (VSS), U2.4 (~{CE}), U2.5 (EN2), U2.8 (VSS), Y1.2, Y2.2
- net at U1.C1 (DEC1): now also C6.1
- net at U1.D2 (XL1/P0.00): now also C23.2, Y2.3
- net at U1.D23 (DEC3): now also C7.1
- net at U1.F2 (XL2/P0.01): now also C22.2, Y2.1
- net at U1.H23 (ANT): now also C21.1, L4.2
- net at U1.N24 (DEC5): now also C8.1
- net VDDH: now reaches U1.Y2 (VDDH)
- net VDDH: now also C19.1, C2.1, R3.2, U2.10 (OUT), U2.11 (OUT), U2.6 (EN1)
- new net: J1.A5 (CC1), R1.1
- new net: R4.1, U2.1 (TS)
- new net: R5.2, U2.16 (ISET)
- new net: C20.2, U2.2 (BAT), U2.3 (BAT)
- new net: RED1.1 (K), U2.9 (~{CHG})
- new net: L1.1, L2.2
- new net: J1.A4 (VBUS), J1.A9 (VBUS), J1.B4 (VBUS), J1.B9 (VBUS)
- new net: J1.B5 (CC2), R2.1
- new net: R3.1, RED1.2 (A)
- new net ANTENNA: C14.1, C15.1, L4.1
- no-connect marks 0 -> 7
Other:
- note added: "001"
- note added: "Battery Charging"
- note added: "BenBoard"
- note added: "July 2023"
- note added: "NRF"
- note added: "USB-C"
- note added: "[x] Optional 32kHz on X1/2"
- moved on the sheet: U1

Commit message: awesome
Connections:
- net GND: now also C20.2; no longer C20.1
- net VBUS: now also J1.A4 (VBUS), J1.A9 (VBUS), J1.B4 (VBUS), J1.B9 (VBUS)
- net VBAT: now reaches U2.2 (BAT), U2.3 (BAT)
- net VBAT: now also C20.1; no longer C20.2
Other:
- moved on the sheet: C20
Changed lines of the file:
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@@
   (junction (at 184.15 41.91) (diameter 0) (color 0 0 0 0)
   )
+  (junction (at 219.71 64.77) (diameter 0) (color 0 0 0 0)
+  )
   (junction (at 128.27 87.63) (diameter 0) (color 0 0 0 0)
   )
@@
   )
   (junction (at 87.63 35.56) (diameter 0) (color 0 0 0 0)
-  )
-  (junction (at 226.06 64.77) (diameter 0) (color 0 0 0 0)
   )
   (no_connect (at 171.45 72.39))
@@
     (stroke (width 0) (type default))
   )
-  (wire (pts (xy 201.93 64.77) (xy 217.17 64.77))
+  (wire (pts (xy 201.93 64.77) (xy 219.71 64.77))
     (stroke (width 0) (type default))
   )
@@
     (stroke (width 0) (type default))
   )
-  (wire (pts (xy 224.79 64.77) (xy 226.06 64.77))
-    (stroke (width 0) (type default))
-  )
   (wire (pts (xy 287.02 48.26) (xy 287.02 50.8))
     (stroke (width 0) (type default))
@@
     (stroke (width 0) (type default))
   )
+  (wire (pts (xy 219.71 64.77) (xy 227.33 64.77))
+    (stroke (width 0) (type default))
+  )
   (wire (pts (xy 60.96 73.66) (xy 62.23 73.66))
     (stroke (width 0) (type default))
@@
     (stroke (width 0) (type default))
   )
-  (wire (pts (xy 226.06 64.77) (xy 227.33 64.77))
-    (stroke (width 0) (type default))
-  )
   (wire (pts (xy 175.26 41.91) (xy 173.99 41.91))
     (stroke (width 0) (type default))
@@
     (stroke (width 0) (type default))
   )
-  (wire (pts (xy 226.06 64.77) (xy 226.06 66.04))
-    (stroke (width 0) (type default))
-  )
   (wire (pts (xy 170.18 74.93) (xy 171.45 74.93))
     (stroke (width 0) (type default))
@@
     (stroke (width 0) (type default))
   )
+  (wire (pts (xy 219.71 73.66) (xy 219.71 72.39))
+    (stroke (width 0) (type default))
+  )
   (wire (pts (xy 115.57 118.11) (xy 116.84 118.11))
+    (stroke (width 0) (type default))
+  )
+  (wire (pts (xy 270.51 43.18) (xy 271.78 43.18))
     (stroke (width 0) (type default))
   )
@@
     )
   )
-  (symbol (lib_id "Device:C") (at 220.98 64.77 270) (unit 1)
-    (in_bom yes) (on_board yes) (dnp no)
-    (property "Reference" "C20" (at 220.98 71.12 90)
-      (effects (font (size 1.27 1.27)))
-    )
-    (property "Value" "4.7uF" (at 220.98 68.58 90)
-      (effects (font (size 1.27 1.27)))
-    )
-    (property "Footprint" "Capacitor_SMD:C_0603_1608Metric" (at 217.17 65.7352 0)
-      (effects (font (size 1.27 1.27)) hide)
-    )
-    (property "Datasheet" "~" (at 220.98 64.77 0)
+  (symbol (lib_id "Device:C") (at 219.71 68.58 0) (unit 1)
+    (in_bom yes) (on_board yes) (dnp no)
+    (property "Reference" "C20" (at 226.06 68.58 90)
+      (effects (font (size 1.27 1.27)))
+    )
+    (property "Value" "4.7uF" (at 223.52 68.58 90)
+      (effects (font (size 1.27 1.27)))
+    )
+    (property "Footprint" "Capacitor_SMD:C_0603_1608Metric" (at 220.6752 72.39 0)
+      (effects (font (size 1.27 1.27)) hide)
+    )
+    (property "Datasheet" "~" (at 219.71 68.58 0)
       (effects (font (size 1.27 1.27)) hide)
     )
@@
     )
   )
-  (symbol (lib_id "power:GND") (at 226.06 66.04 0) (unit 1)
-    (in_bom yes) (on_board yes) (dnp no)
-    (property "Reference" "#PWR018" (at 226.06 72.39 0)
-      (effects (font (size 1.27 1.27)) hide)
-    )
-    (property "Value" "GND" (at 226.06 69.85 0)
-      (effects (font (size 1.27 1.27)))
-    )
-    (property "Footprint" "" (at 226.06 66.04 0)
-      (effects (font (size 1.27 1.27)) hide)
-    )
-    (property "Datasheet" "" (at 226.06 66.04 0)
-      (effects (font (size 1.27 1.27)) hide)
-    )
+  (symbol (lib_id "power:GND") (at 219.71 73.66 0) (unit 1)
+    (in_bom yes) (on_board yes) (dnp no)
+    (property "Reference" "#PWR018" (at 219.71 80.01 0)
+      (effects (font (size 1.27 1.27)) hide)
+    )
+    (property "Value" "GND" (at 219.71 77.47 0)
+      (effects (font (size 1.27 1.27)))
+    )
+    (property "Footprint" "" (at 219.71 73.66 0)
+      (effects (font (size 1.27 1.27)) hide)
+    )
+    (property "Datasheet" "" (at 219.71 73.66 0)
+      (effects (font (size 1.27 1.27)) hide)
+    )

Commit message: epic
Parts:
- removed C15: 100pF, Capacitor_SMD:C_0603_1608Metric, symbol Device:C
- C14: value 100pF -> 0.5pF
- C21: value 100pF -> 0.8pF
- L4: value 3.9nH -> 4.1nH
- SW1: footprint keyswitches:Kailh_socket_MX_optional_reversible -> keyswitches:Kailh_socket_MX
Connections:
- net GND: now also J1.S1 (SHIELD), SW1.1, SW1.1, SW1.1, SW1.1, SW1.1, SW1.1, SW1.1, SW1.1, SW1.1, SW1.1, SW1.1, SW1.1, SW1.1, SW1.1, SW1.1, SW1.1, SW1.1, SW1.1, SW1.1, SW1.1, SW1.1
- net SW2: now reaches SW1.2
- net SW2: now also U1.AC15 (P0.19)
- net SW1: now reaches SW1.2
- net SW1: now also U1.AD10 (P0.15)
- net SW16: now reaches SW1.2
- net SW16: now also U1.W24 (P1.02)
- net SW4: now reaches SW1.2
- net SW4: now also U1.AD12 (P0.17)
- net SW10: now reaches SW1.2
- net SW10: now also U1.AD18 (P0.22)
- net SW9: now reaches SW1.2
- net SW9: now also U1.L1 (P0.06)
- net SW14: now reaches SW1.2
- net SW14: now also U1.AD22 (TRACEDATA0/P1.00)
- net SW7: now reaches SW1.2
- net SW7: now also U1.AD16 (P0.20)
- net SW18: now reaches SW1.2
- net SW18: now also U1.R24 (P1.06)
- net SW15: now reaches SW1.2
- net SW15: now also U1.P23 (P1.07)
- net SW17: now reaches SW1.2
- net SW17: now also U1.U24 (P1.04)
- net SW11: now reaches SW1.2
- net SW11: now also U1.AC21 (P0.25)
- net SW5: now reaches U1.AC17 (P0.21)
- net SW5: now also SW1.2
- net SW8: now reaches U1.AC19 (P0.23)
- net SW8: now also SW1.2
- net SW13: now reaches U1.AD20 (P0.24)
- net SW13: now also SW1.2
- net SW12: now reaches U1.H2 (P0.27)
- net SW12: now also SW1.2
- net SW6: now reaches U1.N1 (P0.08)
- net SW6: now also SW1.2
- net SW3: now reaches U1.P2 (P1.08)
- net SW3: now also SW1.2
- net SW21: now reaches U1.T23 (P1.05)
- net SW21: now also SW1.2
- net SW20: now reaches U1.V23 (P1.03)
- net SW20: now also SW1.2
- net SW19: now reaches U1.Y23 (P1.01)
- net SW19: now also SW1.2
- no-connect marks 7 -> 6
Other:
- note added: "Ben Labs Ltd."
- note added: "Switches"
- note added: "[x] Optional 32kHz on X1/2 [ ] Figure out VDD"
- note removed: "[x] Optional 32kHz on X1/2"
- moved on the sheet: SW1
