File: PID Toaster/PID Toaster.kicad_sch (KiCad schematic)
At the start: 3 parts, among them U1 RP2350A-QFN60, U2 MAX31855KASA, U3 MAX31855KASA

Commit message: toaster
Parts:
- removed U3: MAX31855KASA, Package_SO:SOIC-8_3.9x4.9mm_P1.27mm, symbol Sensor_Temperature:MAX31855KASA
- added C1, C2, C3, C7: 4.7uF, Capacitor_SMD:C_0805_2012Metric_Pad1.18x1.45mm_HandSolder, symbol Device:C
- added C10, C11, C12, C13, C14, C15, C16, C17, C18, C24, C6, C8, C9: 100nF, Capacitor_SMD:C_0805_2012Metric_Pad1.18x1.45mm_HandSolder, symbol Device:C
- added C19: 10uF, Capacitor_SMD:CP_Elec_5x4.4, symbol Device:C_Polarized
- added C20, C22, C23, C27, C28: 10uF, Capacitor_SMD:C_0805_2012Metric_Pad1.18x1.45mm_HandSolder, symbol Device:C
- added C21: 22uF, Capacitor_SMD:C_0805_2012Metric_Pad1.18x1.45mm_HandSolder, symbol Device:C
- added C25, C26: 0.1uF, Capacitor_SMD:C_0805_2012Metric_Pad1.18x1.45mm_HandSolder, symbol Device:C
- added C4, C5: 15pF, Capacitor_SMD:C_0805_2012Metric_Pad1.18x1.45mm_HandSolder, symbol Device:C
- added D1: LED, LED_SMD:LED_0805_2012Metric_Pad1.15x1.40mm_HandSolder, symbol Device:LED
- added D10, D11, D12, D13, D14, D15, D16, D17, D18, D19, D20, D5, D6, D7, D8, D9: D, Diode_SMD:D_0805_2012Metric_Pad1.15x1.40mm_HandSolder, symbol Device:D
- added D2, D3, D4: D, Diode_SMD:D_2010_5025Metric, symbol Device:D
- added J1, J3, J7, J8: Conn_01x02_Socket, Connector_Phoenix_MSTB:PhoenixContact_MSTBA_2,5_2-G-5,08_1x02_P5.08mm_Horizontal, symbol Connector:Conn_01x02_Socket
- added J2, J5: Conn_01x03_Socket, Connector:FanPinHeader_1x03_P2.54mm_Vertical, symbol Connector:Conn_01x03_Socket
- added J4: AVR-JTAG-10, Connector_PinHeader_1.27mm:PinHeader_2x05_P1.27mm_Vertical, symbol Connector:AVR-JTAG-10
- added J6: Conn_01x08_Socket, Connector_JST:JST_PH_S8B-PH-K_1x08_P2.00mm_Horizontal, symbol Connector:Conn_01x08_Socket
- added J9: Micro_SD_Card, Connector_Card:microSD_HC_Hirose_DM3AT-SF-PEJM5, symbol Connector:Micro_SD_Card
- added L1: 3.3uH, Inductor_SMD:L_0603_1608Metric_Pad1.05x0.95mm_HandSolder, symbol Device:L
- added P1: USB_C_Plug_USB2.0, Connector_USB:USB_C_Receptacle_GCT_USB4105-xx-A_16P_TopMnt_Horizontal, symbol Connector:USB_C_Plug_USB2.0
- added PS1: IRM-02-12, Converter_ACDC:Converter_ACDC_MeanWell_IRM-02-xx_THT, symbol Converter_ACDC:IRM-02-12
- added Q1, Q3: NPN, Package_TO_SOT_SMD:SOT-23, symbol Simulation_SPICE:NPN
- added Q2, Q4: PNP, Package_TO_SOT_SMD:SOT-23, symbol Simulation_SPICE:PNP
- added R1, R7: 5k, Resistor_SMD:R_0805_2012Metric_Pad1.20x1.40mm_HandSolder, symbol Device:R
- added R10: 150, Resistor_SMD:R_0805_2012Metric_Pad1.20x1.40mm_HandSolder, symbol Device:R
- added R11, R3, R4, R5, R6: 1k, Resistor_SMD:R_0805_2012Metric_Pad1.20x1.40mm_HandSolder, symbol Device:R
- added R12, R13, R14, R15, R16: 10k, Resistor_SMD:R_0805_2012Metric_Pad1.20x1.40mm_HandSolder, symbol Device:R
- added R2: 33, Resistor_SMD:R_0805_2012Metric_Pad1.20x1.40mm_HandSolder, symbol Device:R
- added R8, R9: 27, Resistor_SMD:R_0805_2012Metric_Pad1.20x1.40mm_HandSolder, symbol Device:R
- added SW1, SW2: SW_Push, Button_Switch_SMD:SW_Push_1P1T_XKB_TS-1187A, symbol Switch:SW_Push
- added SW10, SW11, SW12, SW13, SW14, SW15, SW16, SW17, SW18, SW3, SW4, SW5, SW6, SW7, SW8, SW9: SW_Push, Button_Switch_Keyboard:SW_Cherry_MX_1.00u_PCB, symbol Switch:SW_Push
- added U1: W25Q128JVS, Package_SO:SOIC-8_5.3x5.3mm_P1.27mm, symbol Memory_Flash:W25Q128JVS
- added U3: AMS1117, Package_TO_SOT_SMD:SOT-223-3_TabPin2, symbol Regulator_Linear:AMS1117
- added U4: NCP1117-3.3_SOT223, Package_TO_SOT_SMD:SOT-223-3_TabPin2, symbol Regulator_Linear:NCP1117-3.3_SOT223
- added U6: MAX31855KASA, Package_SO:SOIC-8_3.9x4.9mm_P1.27mm, symbol Sensor_Temperature:MAX31855KASA
- added Y1: 12MHz, Crystal:Crystal_SMD_Abracon_ABM8G-4Pin_3.2x2.5mm, symbol Device:Crystal_GND24_Small
- U2: renamed from U1; footprint (none) -> Toaster:RP2350A_QFN-60_EP_7.75x7.75_Pitch0.4mm
- renumbered U2 to U5
Connections:
- net +3V3: now reaches U2.1 (IOVDD)
- net +3V3: now also U2.11 (IOVDD), U2.20 (IOVDD), U2.30 (IOVDD), U2.38 (IOVDD), U2.44 (ADC_AVDD), U2.45 (IOVDD), U2.49 (VREG_VIN), U2.53 (USB_OTP_VDD), U2.54 (QSPI_IOVDD), U5.4 (V_{CC}), C1.1, C11.1, C12.1, C13.1, C14.1, C16.1, C17.1, C18.1, C23.1, C24.1, C27.1, C28.1, C9.1, D4.1 (K), J6.1 (Pin_1), J9.4 (VDD), R12.2, R13.2, R14.2, R15.2, R2.2, U1.8 (VCC), U6.4 (V_{CC})
- net KEYPAD_COL_1: now reaches U2.10 (GPIO7)
- net KEYPAD_COL_1: now also SW10.1, SW7.1, SW8.1, SW9.1
- net KEYPAD_COL_2: now reaches U2.12 (GPIO8)
- net KEYPAD_COL_2: now also SW11.1, SW12.1, SW13.1, SW14.1
- net KEYPAD_COL_3: now reaches U2.13 (GPIO9)
- net KEYPAD_COL_3: now also SW15.1, SW16.1, SW17.1, SW18.1
- net KEYPAD_ROW_0: now reaches U2.14 (GPIO10)
- net KEYPAD_ROW_0: now also D13.1 (K), D17.1 (K), D5.1 (K), D9.1 (K)
- net KEYPAD_ROW_1: now reaches U2.15 (GPIO11)
- net KEYPAD_ROW_1: now also D10.1 (K), D14.1 (K), D18.1 (K), D6.1 (K)
- net KEYPAD_ROW_2: now reaches U2.16 (GPIO12)
- net KEYPAD_ROW_2: now also D11.1 (K), D15.1 (K), D19.1 (K), D7.1 (K)
- net KEYPAD_ROW_3: now reaches U2.17 (GPIO13)
- net KEYPAD_ROW_3: now also D12.1 (K), D16.1 (K), D20.1 (K), D8.1 (K)
- net USR_PWM_0: now reaches U2.18 (GPIO14)
- net USR_PWM_0: now also R1.1
- net USR_PWM_0_AUX: now reaches U2.19 (GPIO15)
- net USR_PWM_0_AUX: now also J2.1 (Pin_1)
- net SPI_THERMAL_2_CS: now reaches U2.2 (GPIO0)
- net SPI_THERMAL_2_CS: now also U6.6 (~{CS})
- net at U2.21 (XIN): now also C4.2, Y1.1
- net at U2.22 (XOUT): now also R6.2
- net +1V1: now reaches U2.23 (DVDD)
- net +1V1: now also U2.39 (DVDD), U2.50 (VREG_FB), U2.6 (DVDD), C10.1, C2.1, C7.1, C8.1, L1.1
- net SWCLK: now reaches U2.24 (SWCLK)
- net SWCLK: now also J4.1 (TCK)
- net SWIO: now reaches U2.25 (SWDIO)
- net SWIO: now also J4.5 (TMS)
- net RESET: now reaches U2.26 (RUN)
- net RESET: now also J4.6 (~{SRST}), R5.1
- net USR_PWM_1: now reaches U2.27 (GPIO16)
- net USR_PWM_1: now also R7.1
- net USR_PWM_1_AUX: now reaches U2.28 (GPIO17)
- net USR_PWM_1_AUX: now also J5.1 (Pin_1)
- net SSR_SWITCH: now reaches U2.29 (GPIO18)
- net SSR_SWITCH: now also J1.2 (Pin_2)
- net SPI_THERMAL_1_CS: now reaches U2.3 (GPIO1)
- net SPI_THERMAL_1_CS: now also U5.6 (~{CS})
- net DISPLAY_SPI_MOSI: now reaches U2.31 (GPIO19)
- net DISPLAY_SPI_MOSI: now also J6.3 (Pin_3)
- net DISPLAY_SPI_SCK: now reaches U2.32 (GPIO20)
- net DISPLAY_SPI_SCK: now also J6.4 (Pin_4)
- net DISPLAY_SPI_CS: now reaches U2.33 (GPIO21)
- net DISPLAY_SPI_CS: now also J6.5 (Pin_5)
- net DISPLAY_SPI_DS: now reaches U2.34 (GPIO22)
- net DISPLAY_SPI_DS: now also J6.6 (Pin_6)
- net DISPLAY_RST: now reaches U2.35 (GPIO23)
- net DISPLAY_RST: now also J6.7 (Pin_7)
- net DISPLAY_BL: now reaches U2.36 (GPIO24)
- net DISPLAY_BL: now also J6.8 (Pin_8)
- net at U2.37 (GPIO25): now also R10.1
- net SPI_SD_CS: now reaches U2.4 (GPIO2)
- net SPI_SD_CS: now also J9.2 (DAT3/CD), R12.1
- net at U2.46 (VREG_AVDD): now also C3.1, R2.1
- net GND: now reaches U2.47 (VREG_PGND)
- net GND: now also U2.61 (GND), U5.1 (GND), C1.2, C10.2, C11.2, C12.2, C13.2, C14.2, C15.2, C16.2, C17.2, C18.2, C19.2, C2.2, C20.2, C21.2, C22.2, C23.2, C24.2, C27.2, C28.2, C3.2, C4.1, C5.2, C6.2, C7.2, C8.2, C9.2, D1.1 (K), J1.1 (Pin_1), J2.3 (Pin_3), J4.10 (GND), J4.2 (GND), J5.3 (Pin_3), J6.2 (Pin_2), J9.6 (VSS), P1.A1 (GND), P1.A12 (GND), P1.B1 (GND), P1.B12 (GND), P1.S1 (SHIELD), PS1.3 (-Vo), Q1.3 (E), Q3.3 (E), SW1.1, SW2.1, U1.4 (GND), U3.1 (ADJ), U4.1 (GND), U6.1 (GND), Y1.2, Y1.4
- net at U2.48 (VREG_LX): now also L1.2
- net SPI_MISO: now reaches U2.5 (GPIO3)
- net SPI_MISO: now also J9.7 (DAT0), R15.1
- net at U2.51 (USB_DM): now also R9.1
- net at U2.52 (USB_DP): now also R8.2
- net QSPI_SD3: now reaches U2.55 (QSPI_SD3)
- net QSPI_SD3: now also U1.7 (~{HOLD}/~{RESET}/IO_{3})
- net QSPI_SDCLK: now reaches U2.56 (QSPI_SCLK)
- net QSPI_SDCLK: now also U1.6 (CLK)
- net QSPI_SD0: now reaches U2.57 (QSPI_SD0)
- net QSPI_SD0: now also U1.5 (DI/IO_{0})
- net QSPI_SD2: now reaches U2.58 (QSPI_SD2)
- net QSPI_SD2: now also U1.3 (~{WP}/IO_{2})
- net QSPI_SD1: now reaches U2.59 (QSPI_SD1)
- net QSPI_SD1: now also U1.2 (DO/IO_{1})
- net QSPI_SS: now reaches U2.60 (QSPI_SS)
- net QSPI_SS: now also R3.1, U1.1 (~{CS})
- net SPI_MOSI: now reaches U2.7 (GPIO4)
- net SPI_MOSI: now also J9.3 (CMD), R13.1
- net SPI_SCK: now reaches U2.8 (GPIO5)
- net SPI_SCK: now also J9.5 (CLK), R14.1
- net KEYPAD_COL_0: now reaches U2.9 (GPIO6)
- net KEYPAD_COL_0: now also SW3.1, SW4.1, SW5.1, SW6.1
- net at U5.2 (T-): now also C25.2, J7.1 (Pin_1)
- net at U5.3 (T+): now also C25.1, J7.2 (Pin_2)
- net SPI_THERMAL_SCK: now reaches U5.5 (SCK)
- net SPI_THERMAL_SCK: now also U6.5 (SCK)
- net SPI_THERMAL_MISO: now reaches U5.7 (SO)
- net SPI_THERMAL_MISO: now also U6.7 (SO)
- new net: D19.2 (A), SW17.2
- new net: D8.2 (A), SW6.2
- new net: D9.2 (A), SW7.2
- new net: D11.2 (A), SW9.2
- new net: C15.1, Q3.1 (C), R11.2
- new net: J2.2 (Pin_2), Q2.1 (C)
- new net: Q2.2 (B), R4.1
- new net: D18.2 (A), SW16.2
- new net: D14.2 (A), SW12.2
- new net: C22.1, D4.2 (A), U4.2 (VO)
- new net: D1.2 (A), R10.2
- new net: J3.1 (Pin_1), PS1.1 (AC/N)
- new net: J3.2 (Pin_2), PS1.2 (AC/L)
- new net: D20.2 (A), SW18.2
- new net: R3.2, SW1.2
- new net: D7.2 (A), SW5.2
- new net: C5.1, R6.1, Y1.3
- new net: C6.1, Q1.1 (C), R4.2
- new net: Q1.2 (B), R1.2
- new net: D12.2 (A), SW10.2
- new net: C21.1, D3.2 (A), U3.2 (VO)
- new net: R5.2, SW2.2
- new net: C26.1, J8.2 (Pin_2), U6.3 (T+)
- new net: C26.2, J8.1 (Pin_1), U6.2 (T-)
- new net: Q3.2 (B), R7.2
- new net: D16.2 (A), SW14.2
- new net: D13.2 (A), SW11.2
- new net: D10.2 (A), SW8.2
- new net: Q4.2 (B), R11.1
- new net: P1.A5 (CC), R16.1
- new net: J5.2 (Pin_2), Q4.1 (C)
- new net: D6.2 (A), SW4.2
- new net: D17.2 (A), SW15.2
- new net: D5.2 (A), SW3.2
- new net: D15.2 (A), SW13.2
- new net +12V: C19.1, PS1.4 (+Vo), Q2.3 (E), Q4.3 (E), U3.3 (VI)
- new net +5V: C20.1, D2.1 (K), D3.1 (K), U4.3 (VI)
- new net D+: P1.A6 (D+), R8.1
- new net D-: P1.A7 (D-), R9.2
- new net VBUS: D2.2 (A), J4.4 (VREF), J4.7 (VCC), P1.A4 (VBUS), P1.A9 (VBUS), P1.B4 (VBUS), P1.B9 (VBUS), R16.2
- no-connect marks 0 -> 10
Other:
- note added: "CONN"
- note added: "DISPLAY"
- note added: "FAN CONTROL"
- note added: "HVAC"
- note added: "KEYPAD"
- note added: "POWER"
- note added: "RP2350"
- note added: "RP2350 AUX"
- note added: "SD"
- note added: "THERMOCOUPLE"
- company: (none) -> Ben Labs
- title: (none) -> PID Controlled Oven
- moved on the sheet: U2, U5
