File: HDD Backplane/HDD Backplane.kicad_pcb (KiCad board)
At the start: 2 copper layers, 205 x 133 mm, 28 parts, among them J1 SATA_COMBINED_22, J13 Conn_01x04_Pin, J14 Conn_01x04_Pin, J7 SATA_DATA_7

Commit message: Backplane
Parts:
- removed D1 (x6): LED, LED_SMD:LED_0805_2012Metric_Pad1.15x1.40mm_HandSolder
- renumbered J1 to J10, J1 to J12, J1 to J2, J1 to J3, J1 to J5
Connections:
- J1 pad 18: /s1_act -> GND
- J1 pad 8: unconnected-(J1-V3.3-Pad8) -> GND
- J1 pad 9: unconnected-(J1-V3.3-Pad9) -> GND
- J10 pad 18: /s1_act -> GND
- J10 pad 8: unconnected-(J1-V3.3-Pad8) -> GND
- J10 pad 9: unconnected-(J1-V3.3-Pad9) -> GND
- J12 pad 18: /s1_act -> GND
- J12 pad 8: unconnected-(J1-V3.3-Pad8) -> GND
- J12 pad 9: unconnected-(J1-V3.3-Pad9) -> GND
- J2 pad 18: /s1_act -> GND
- J2 pad 8: unconnected-(J1-V3.3-Pad8) -> GND
- J2 pad 9: unconnected-(J1-V3.3-Pad9) -> GND
- J3 pad 18: /s1_act -> GND
- J3 pad 8: unconnected-(J1-V3.3-Pad8) -> GND
- J3 pad 9: unconnected-(J1-V3.3-Pad9) -> GND
- J5 pad 18: /s1_act -> GND
- J5 pad 8: unconnected-(J1-V3.3-Pad8) -> GND
- J5 pad 9: unconnected-(J1-V3.3-Pad9) -> GND
Routing:
- net /s1_act: track 72.3 -> 0.00 mm
- net GND: track 25.2 -> 25.3 mm, vias 4 -> 0
- added copper zone on B.Cu, net +5V
- added copper zone on F.Cu, net +5V
Other:
- board text added: "+12v"
- board text added: "+5v"
- board text added: "GND"
