File: HDD Backplane/HDD Backplane.kicad_sch (KiCad schematic)
At the start: 20 parts, among them J1 SATA_COMBINED_22, J10 SATA_COMBINED_22, J11 SATA_DATA_7, J12 SATA_COMBINED_22, J13 Conn_01x04_Pin, J14 Conn_01x04_Pin, J2 SATA_COMBINED_22, J3 SATA_COMBINED_22, J4 SATA_DATA_7, J5 SATA_COMBINED_22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

Commit message: Backplane
Parts:
- removed D1, D2, D3, D4, D5, D6: LED, LED_SMD:LED_0805_2012Metric_Pad1.15x1.40mm_HandSolder, symbol Device:LED
Connections:
- net s1_act is gone; now on net GND: J1.18 (ACT)
- net s2_act is gone; now on net GND: J2.18 (ACT)
- net s3_act is gone; now on net GND: J3.18 (ACT)
- net s4_act is gone; now on net GND: J5.18 (ACT)
- net s5_act is gone; now on net GND: J10.18 (ACT)
- net s6_act is gone; now on net GND: J12.18 (ACT)
- net GND: now also J1.8 (V3.3), J1.9 (V3.3), J10.8 (V3.3), J10.9 (V3.3), J12.8 (V3.3), J12.9 (V3.3), J2.8 (V3.3), J2.9 (V3.3), J3.8 (V3.3), J3.9 (V3.3), J5.8 (V3.3), J5.9 (V3.3)
- no-connect marks 12 -> 0
